File: esp32/esp32.kicad_pcb (KiCad board)
At the start: 4 copper layers, 151.1 x 100.3 mm, 40 parts, among them J1 USB_B_Micro, J2 Conn_01x02_Male, Q1 S8050, Q2 S8050, U1 ESP32-WROOM-32, U2 NCP1117-3.3_TO252, U3 CP2102N-A01-GQFN28

Commit message: usb routing
Parts:
- removed C16: 0.1uF/25V(10%), Capacitor_SMD:C_0402_1005Metric
- removed C18: 10uF/25V(10%), Capacitor_SMD:C_0603_1608Metric
- removed C23: 10uF/25V(10%)(NC), Capacitor_SMD:C_0402_1005Metric
- removed the D4 at (223.0, 104.0)
- removed R15: 5K(1%)(NC), Resistor_SMD:R_0402_1005Metric
- removed R24: 0R(1%), Resistor_SMD:R_0402_1005Metric
- removed R25: 3.3K(1%)(NC), Resistor_SMD:R_0402_1005Metric
- removed the R7 at (236.0, 117.0)
- added D3: ESD05V88D-LC, Diode_SMD:D_SOD-923, F.Cu at (127.4, 79.6)
- added D5: ESD05V88D-LC, Diode_SMD:D_SOD-923, F.Cu at (125.4, 79.6)
- added J3: Conn_01x19_Pin, Connector_PinHeader_1.00mm:PinHeader_1x19_P1.00mm_Vertical, F.Cu at (139.2, 38.5)
- added R10: 2K(5%), Resistor_SMD:R_0402_1005Metric, F.Cu at (146.8, 75.7)
- added R8: 22.1K(1%), Resistor_SMD:R_0402_1005Metric, F.Cu at (146.8, 71.8)
- added R9: 47.5K(1%), Resistor_SMD:R_0402_1005Metric, F.Cu at (146.8, 73.7)
- C1: value 10uF/25V(10%) -> 22uF/25V(10%)
- C5: renamed from C15; value 1nF/50V(10%) -> 0.1uF/50V(10%)
- C6: renamed from C9; value 1nF/50V(10%) -> 0.1uF/50V(10%)
- C7: renamed from C14; value 1nF/50V(10%) -> 0.1uF/50V(10%)
- C8: renamed from C21; value 100uF/6.3V(20%) -> 22uF/10V(20%)
- C9: renamed from C22; value 1uF/10V(10%) -> 0.1uF/50V(10%)
- D2: footprint Diode_SMD:D_0402_1005Metric -> Diode_SMD:D_SOD-923
- J2: value Conn_01x02_Male -> Conn_01x19_Pin; footprint Connector_JST:JST_EH_B2B-EH-A_1x02_P2.50mm_Vertical -> Connector_PinHeader_1.00mm:PinHeader_1x19_P1.00mm_Vertical
- R13: renamed from R12; value 12K(1%) -> 10K(5%)
- moved U3 140.7 mm to (126.5, 47.5)
- moved J2 122.2 mm to (113.8, 38.5), turned to 0 degrees
- moved Reset1 115.3 mm to (117.4, 82.0), turned to -90 degrees
- moved Q1 111.8 mm to (136.5, 64.5), turned to 90 degrees
- moved U1 109.9 mm to (127.0, 64.4)
- moved U2 109.4 mm to (126.6, 74.0), turned to -90 degrees
- moved C8 108.0 mm to (114.5, 65.0)
- moved C9 108.0 mm to (115.5, 61.0)
- moved J1 107.3 mm to (126.5, 83.7)
- moved Q2 105.8 mm to (136.5, 74.2), turned to -90 degrees
- moved D2 105.5 mm to (122.8, 80.0)
- moved D1 105.0 mm to (119.8, 66.2), turned to -90 degrees
- moved C2 104.9 mm to (121.0, 63.2), turned to 90 degrees
- moved C3 103.3 mm to (122.0, 71.0)
- moved C4 101.2 mm to (122.0, 72.2), turned to 180 degrees
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- renumbered C3 to C2, C20 to C3, C19 to C4, D3 to D4, R2 to R1, R23 to R11, R3 to R12, R4 to R14, R17 to R2, R18 to R3, R19 to R4, R20 to R5, R21 to R6, R22 to R7, U2 to U1, U3 to U2, U1 to U3
Connections:
- D2 pad 1: USB_DP -> VBUS
- D4 pad 2: Net-(D3-Pad2) -> VBUS
- J1 pad 1: Net-(D3-Pad2) -> VBUS
- J1 pad 4: Net-(J1-Pad4) -> unconnected-(J1-ID-Pad4)
- J2 pad 1: +5V -> +3V3
- J2 pad 2: GND -> EN
- U1 pad 1: Net-(C23-Pad1) -> GND
- U2 pad 10: Net-(U3-Pad10) -> unconnected-(U2-NC-Pad10)
- U2 pad 12: Net-(U3-Pad12) -> unconnected-(U2-SUSPEND-Pad12)
- U2 pad 13: Net-(U3-Pad13) -> unconnected-(U2-CHREN-Pad13)
- U2 pad 14: Net-(U3-Pad14) -> unconnected-(U2-CHR1-Pad14)
- U2 pad 15: Net-(U3-Pad15) -> unconnected-(U2-CHR0-Pad15)
- U2 pad 16: Net-(U3-Pad16) -> unconnected-(U2-~{WAKEUP}/GPIO.3-Pad16)
- U2 pad 17: Net-(U3-Pad17) -> unconnected-(U2-RS485/GPIO.2-Pad17)
- U2 pad 18: Net-(U3-Pad18) -> unconnected-(U2-~{RXT}/GPIO.1-Pad18)
- U2 pad 19: Net-(U3-Pad19) -> unconnected-(U2-~{TXT}/GPIO.0-Pad19)
- U2 pad 20: Net-(U3-Pad20) -> unconnected-(U2-GPIO.6-Pad20)
- U2 pad 21: Net-(U3-Pad21) -> unconnected-(U2-GPIO.5-Pad21)
- U2 pad 22: Net-(U3-Pad22) -> unconnected-(U2-GPIO.4-Pad22)
- U2 pad 8: +5V -> Net-(U2-VBUS)
- U3 pad 32: Net-(U1-Pad32) -> unconnected-(U3-NC-Pad32)
Routing:
- net USB_DN: track 0.00 -> 18.4 mm, vias 0 -> 2
- net USB_DP: track 0.00 -> 17.5 mm, vias 0 -> 2
- net VBUS: track 0.00 -> 3.55 mm
- removed copper zone on Vdd, net +3V3
- removed copper zone on Gnd, net GND
Other:
- board size 151.1 x 100.3 mm -> 27.9 x 48.2 mm
- copper layers 4 -> 2
- net class Default removed
