File: esp32/esp32.kicad_sch (KiCad schematic)
At the start: 38 parts, among them J1 USB_B_Micro, Q1 S8050, Q2 S8050, U1 ESP32-WROOM-32, U2 NCP1117-3.3_TO252, U3 CP2102N-A01-GQFN28

Commit message: usb routing
Parts:
- removed D4: ESD05V88D-LC, Diode_SMD:D_0402_1005Metric, symbol esp32-rescue:ESD9B5.0ST5G-Diode
- added D5: ESD05V88D-LC, Diode_SMD:D_SOD-923, symbol esp32-rescue:ESD9B5.0ST5G-Diode
- D2, D3: renamed from D?; footprint Diode_SMD:D_0402_1005Metric -> Diode_SMD:D_SOD-923
- gave numbers to parts that had none: 6
- renumbered C3 to C2, C20 to C3, C19 to C4, C15 to C5, C9 to C6, C14 to C7, C21 to C8, C22 to C9, D3 to D4, R2 to R1, R23 to R11, R3 to R12, R12 to R13, R4 to R14, R17 to R2, R18 to R3, R19 to R4, R20 to R5, R21 to R6, R22 to R7, U2 to U1, U3 to U2, U1 to U3
Connections:
- net GND: now also D5.2 (A2)
- net USB_DN: now also D5.1 (A1)
Other:
- moved on the sheet: Boot1, C1, C2, C3, C4, C5, C6, C7, C8, C9, D1, D2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
